File: VideoBoy1.1eagle/VideoBoy1.12.brd (EAGLE design)
At the start: 101.6 x 86.4 mm, 75 parts, among them IC5 74126PW, IC6 74393AT-PWRQ1, IC7 74126PW, IC8 74126PW, IC9 74126PW, J5 POWERPOLE_POWER25A

Commit message: edited circuit drains
Parts:
- turned J1 to 0 degrees
- turned J2 to 0 degrees
- turned J3 to 0 degrees
- turned J4 to 0 degrees
Connections:
- net DRAIN1: now also J1.4
- net DRAIN2: now also J1.3
- net DRAIN3: now also J2.4
- net DRAIN4: now also J2.3
- net DRAIN5: now also J3.4
- net DRAIN6: now also J3.3
- net DRAIN7: now also J4.4
- net DRAIN8: now also J4.3
- net GND: no longer J1.3, J1.4, J2.3, J2.4, J3.3, J3.4, J4.3, J4.4
Routing:
- net DRAIN2: track 7.07 -> 36.0 mm
- net DRAIN4: track 6.59 -> 33.8 mm
- net DRAIN8: track 6.55 -> 33.8 mm
- net DRAIN7: track 6.56 -> 32.5 mm
- net DRAIN6: track 6.57 -> 32.3 mm
- net DRAIN5: track 6.56 -> 30.8 mm
- net DRAIN3: track 6.55 -> 29.2 mm
- net DRAIN1: track 6.55 -> 28.3 mm
- net VCC: track 702.1 -> 712.1 mm, vias 14 -> 16
- net EN1: track 114.3 -> 119.2 mm, vias 0 -> 2
- net COUT_1: track 38.1 -> 41.6 mm, vias 1 -> 0
- net EN8: track 51.1 -> 53.8 mm
- net DOUT_1: track 40.6 -> 42.3 mm, vias 1 -> 0
- net COUT_7: track 39.4 -> 41.1 mm
- net COUT_5: track 40.5 -> 39.2 mm
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