File: VideoBoy1.1eagle/VideoBoy1.12.sch (EAGLE design)
At the start: 75 parts, among them IC5 74126PW, IC6 74393AT-PWRQ1, IC7 74126PW, IC8 74126PW, IC9 74126PW, J5 POWERPOLE_POWER25A

Commit message: edited circuit drains
Connections:
- net DRAIN1: now also J1.4
- net DRAIN2: now also J1.3
- net DRAIN3: now also J2.4
- net DRAIN4: now also J2.3
- net DRAIN5: now also J3.4
- net DRAIN6: now also J3.3
- net DRAIN7: now also J4.4
- net DRAIN8: now also J4.3
- net GND: no longer J1.3, J1.4, J2.3, J2.4, J3.3, J3.4, J4.3, J4.4
Changed lines of the file:
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@@
 <part name="IC9" library="My TI Chips" deviceset="74*126" device="PW"/>
 <part name="RN8" library="resistor-dil" library_urn="urn:adsk.eagle:library:342" deviceset="4R-N" device="0603-ARV"/>
-<part name="GND22" library="supply1" library_urn="urn:adsk.eagle:library:371" deviceset="GND" device=""/>
 <part name="GND23" library="supply1" library_urn="urn:adsk.eagle:library:371" deviceset="GND" device=""/>
 <part name="GND24" library="supply1" library_urn="urn:adsk.eagle:library:371" deviceset="GND" device=""/>
@@
 <instance part="RN8" gate="C" x="40.64" y="386.08"/>
 <instance part="RN8" gate="D" x="40.64" y="368.3"/>
-<instance part="GND22" gate="1" x="-259.08" y="264.16"/>
 <instance part="GND23" gate="1" x="-309.88" y="309.88"/>
 <instance part="GND24" gate="1" x="-203.2" y="309.88"/>
@@
 </segment>
 <segment>
-<pinref part="J4" gate="G$1" pin="3"/>
-<pinref part="J4" gate="G$1" pin="4"/>
-<wire x1="-269.24" y1="281.94" x2="-266.7" y2="281.94" width="0.1524" layer="91"/>
-<pinref part="J3" gate="G$1" pin="3"/>
-<pinref part="J3" gate="G$1" pin="4"/>
-<wire x1="-269.24" y1="289.56" x2="-266.7" y2="289.56" width="0.1524" layer="91"/>
-<pinref part="J2" gate="G$1" pin="3"/>
-<pinref part="J2" gate="G$1" pin="4"/>
-<wire x1="-269.24" y1="297.18" x2="-266.7" y2="297.18" width="0.1524" layer="91"/>
-<pinref part="J1" gate="G$1" pin="3"/>
-<pinref part="J1" gate="G$1" pin="4"/>
-<wire x1="-269.24" y1="304.8" x2="-266.7" y2="304.8" width="0.1524" layer="91"/>
-<wire x1="-266.7" y1="304.8" x2="-259.08" y2="304.8" width="0.1524" layer="91"/>
-<junction x="-266.7" y="304.8"/>
-<wire x1="-259.08" y1="304.8" x2="-259.08" y2="297.18" width="0.1524" layer="91"/>
-<wire x1="-259.08" y1="297.18" x2="-259.08" y2="289.56" width="0.1524" layer="91"/>
-<wire x1="-259.08" y1="289.56" x2="-259.08" y2="281.94" width="0.1524" layer="91"/>
-<wire x1="-259.08" y1="281.94" x2="-259.08" y2="266.7" width="0.1524" layer="91"/>
-<wire x1="-266.7" y1="297.18" x2="-259.08" y2="297.18" width="0.1524" layer="91"/>
-<junction x="-266.7" y="297.18"/>
-<junction x="-259.08" y="297.18"/>
-<wire x1="-266.7" y1="289.56" x2="-259.08" y2="289.56" width="0.1524" layer="91"/>
-<junction x="-266.7" y="289.56"/>
-<junction x="-259.08" y="289.56"/>
-<wire x1="-266.7" y1="281.94" x2="-259.08" y2="281.94" width="0.1524" layer="91"/>
-<junction x="-266.7" y="281.94"/>
-<junction x="-259.08" y="281.94"/>
-<pinref part="GND22" gate="1" pin="GND"/>
-</segment>
-<segment>
 <wire x1="-203.2" y1="312.42" x2="-203.2" y2="322.58" width="0.1524" layer="91"/>
 <pinref part="F1" gate="G$1" pin="2"/>
@@
 <label x="-261.62" y="393.7" size="1.778" layer="95"/>
 </segment>
+<segment>
+<pinref part="J1" gate="G$1" pin="4"/>
+<wire x1="-266.7" y1="304.8" x2="-254" y2="304.8" width="0.1524" layer="91"/>
+<label x="-259.08" y="304.8" size="1.778" layer="95"/>
+</segment>
 </net>
 <net name="SOURCE2" class="0">
@@
 <wire x1="-266.7" y1="383.54" x2="-251.46" y2="383.54" width="0.1524" layer="91"/>
 </segment>
+<segment>
+<pinref part="J1" gate="G$1" pin="3"/>
+<wire x1="-269.24" y1="304.8" x2="-269.24" y2="302.26" width="0.1524" layer="91"/>
+<wire x1="-269.24" y1="302.26" x2="-254" y2="302.26" width="0.1524" layer="91"/>
+<label x="-259.08" y="302.26" size="1.778" layer="95"/>
+</segment>
 </net>
 <net name="SOURCE3" class="0">
@@
 <label x="-261.62" y="363.22" size="1.778" layer="95"/>
 </segment>
+<segment>
+<pinref part="J2" gate="G$1" pin="3"/>
+<wire x1="-269.24" y1="297.18" x2="-269.24" y2="294.64" width="0.1524" layer="91"/>
+<wire x1="-269.24" y1="294.64" x2="-254" y2="294.64" width="0.1524" layer="91"/>
+<label x="-259.08" y="294.64" size="1.778" layer="95"/>
+</segment>
 </net>
 <net name="DRAIN5" class="0">
@@
 <label x="-261.62" y="353.06" size="1.778" layer="95"/>
 </segment>
+<segment>
+<pinref part="J3" gate="G$1" pin="4"/>
+<wire x1="-266.7" y1="289.56" x2="-254" y2="289.56" width="0.1524" layer="91"/>
+<label x="-259.08" y="289.56" size="1.778" layer="95"/>
+</segment>
 </net>
 <net name="DRAIN6" class="0">
@@
 <label x="-261.62" y="342.9" size="1.778" layer="95"/>
 </segment>
+<segment>
+<pinref part="J3" gate="G$1" pin="3"/>
+<wire x1="-269.24" y1="289.56" x2="-269.24" y2="287.02" width="0.1524" layer="91"/>
+<wire x1="-269.24" y1="287.02" x2="-254" y2="287.02" width="0.1524" layer="91"/>
+<label x="-259.08" y="287.02" size="1.778" layer="95"/>
+</segment>
 </net>
 <net name="DRAIN7" class="0">
@@
 <label x="-261.62" y="332.74" size="1.778" layer="95"/>
 </segment>
+<segment>
+<pinref part="J4" gate="G$1" pin="4"/>
+<wire x1="-266.7" y1="281.94" x2="-254" y2="281.94" width="0.1524" layer="91"/>
+<label x="-259.08" y="281.94" size="1.778" layer="95"/>
+</segment>
 </net>
 <net name="DRAIN8" class="0">
@@
 <label x="-261.62" y="322.58" size="1.778" layer="95"/>
 </segment>
+<segment>
+<pinref part="J4" gate="G$1" pin="3"/>
+<wire x1="-269.24" y1="281.94" x2="-269.24" y2="279.4" width="0.1524" layer="91"/>
+<wire x1="-269.24" y1="279.4" x2="-254" y2="279.4" width="0.1524" layer="91"/>
+<label x="-259.08" y="279.4" size="1.778" layer="95"/>
+</segment>
 </net>
 <net name="DRAIN3" class="0">
@@
 <label x="-261.62" y="373.38" size="1.778" layer="95"/>
 </segment>
-</net>
+<segment>
+<pinref part="J2" gate="G$1" pin="4"/>
+<wire x1="-266.7" y1="297.18" x2="-254" y2="297.18" width="0.1524" layer="91"/>
+<label x="-259.08" y="297.18" size="1.778" layer="95"/>
+</segment>
+</net>
